Commit message: Refactor launch and URDF files for improved robot simulation setup

File: bot_description/urdf/bot.xacro (robot description, xacro)
@@ -148,5 +148,5 @@
   <parent link="base_link"/>
   <child link="right_wheel_link_1"/>
-  <axis xyz="0.0 -1.0 0.0"/>
+  <axis xyz="0.0 1.0 0.0"/>
 </joint>
 <joint name="left_wheel_joint" type="continuous">
@@ -154,5 +154,5 @@
   <parent link="base_link"/>
   <child link="left_wheel_link_1"/>
-  <axis xyz="0.0 -1.0 0.0"/>
+  <axis xyz="0.0 1.0 0.0"/>
 </joint>
 <joint name="caster_wheel_b_joint" type="fixed">

Commit message: physics ok!

File: bot_description/urdf/bot.xacro (robot description, xacro)
@@ -6,4 +6,11 @@
 <xacro:include filename="$(find bot_description)/urdf/camera.xacro" />
 <xacro:include filename="$(find bot_description)/urdf/lidar.xacro" />
+<!-- Root link: KDL does not support inertia on root link -->
+<link name="base_footprint"/>
+<joint name="base_footprint_joint" type="fixed">
+  <parent link="base_footprint"/>
+  <child link="base_link"/>
+  <origin xyz="0 0 0" rpy="0 0 0"/>
+</joint>
 <link name="base_link">
   <inertial>
@@ -28,7 +35,7 @@
 <link name="right_wheel_link_1">
   <inertial>
-    <origin xyz="-1.4135271091344188e-10 -0.028050466348318148 1.225355835798858e-06" rpy="0 0 0"/>
-    <mass value="0.132130981755143"/>
-    <inertia ixx="0.000164" iyy="0.000293" izz="0.000164" ixy="-0.0" iyz="-0.0" ixz="-0.0"/>
+    <origin xyz="-1.4135269981415094e-10 -0.028050466348318148 1.225355835798858e-06" rpy="0 0 0"/>
+    <mass value="0.09525721940487054"/>
+    <inertia ixx="0.000118" iyy="0.000211" izz="0.000118" ixy="-0.0" iyz="-0.0" ixz="-0.0"/>
   </inertial>
   <visual>
@@ -40,7 +47,7 @@
   </visual>
   <collision>
-    <origin xyz="-0.0 0.1425 -0.0546" rpy="0 0 0"/>
+    <origin xyz="0.0 0.0 0.0" rpy="1.5708 0 0"/>
     <geometry>
-      <mesh filename="file://$(find bot_description)/meshes/right_wheel_link_1.stl" scale="0.001 0.001 0.001"/>
+      <cylinder radius="0.0546" length="0.056"/>
     </geometry>
   </collision>
@@ -49,6 +56,6 @@
   <inertial>
     <origin xyz="1.4973146092150716e-11 0.028050466283458836 -1.2262817377928226e-06" rpy="0 0 0"/>
-    <mass value="0.13213095662214813"/>
-    <inertia ixx="0.000164" iyy="0.000293" izz="0.000164" ixy="0.0" iyz="-0.0" ixz="0.0"/>
+    <mass value="0.0952572012857347"/>
+    <inertia ixx="0.000118" iyy="0.000211" izz="0.000118" ixy="0.0" iyz="-0.0" ixz="0.0"/>
   </inertial>
   <visual>
@@ -60,7 +67,7 @@
   </visual>
   <collision>
-    <origin xyz="0.0 -0.1425 -0.0546" rpy="0 0 0"/>
+    <origin xyz="0.0 0.0 0.0" rpy="1.5708 0 0"/>
     <geometry>
-      <mesh filename="file://$(find bot_description)/meshes/left_wheel_link_1.stl" scale="0.001 0.001 0.001"/>
+      <cylinder radius="0.0546" length="0.056"/>
     </geometry>
   </collision>
@@ -68,7 +75,7 @@
 <link name="caster_wheel_b_1">
   <inertial>
-    <origin xyz="0.01999999999999999 -2.634096614519092e-17 -0.012260416666666649" rpy="0 0 0"/>
-    <mass value="0.01798247634914797"/>
-    <inertia ixx="2e-06" iyy="2e-06" izz="2e-06" ixy="0.0" iyz="-0.0" ixz="-0.0"/>
+    <origin xyz="0.01999999999999999 -5.329070518200751e-17 -0.012188268156424566" rpy="0 0 0"/>
+    <mass value="0.017408884194903947"/>
+    <inertia ixx="2e-06" iyy="2e-06" izz="2e-06" ixy="-0.0" iyz="-0.0" ixz="0.0"/>
   </inertial>
   <visual>
@@ -80,7 +87,7 @@
   </visual>
   <collision>
-    <origin xyz="0.1675 0.0 -0.0291" rpy="0 0 0"/>
+    <origin xyz="0.0 0.0 0.0" rpy="0 0 0"/>
     <geometry>
-      <mesh filename="file://$(find bot_description)/meshes/caster_wheel_b_1.stl" scale="0.001 0.001 0.001"/>
+      <sphere radius="0.028"/>
     </geometry>
   </collision>
@@ -88,7 +95,7 @@
 <link name="caster_wheel_a_1">
   <inertial>
-    <origin xyz="-0.019999999999999962 3.769546289141946e-17 -0.012260416666666652" rpy="0 0 0"/>
-    <mass value="0.01798247634914797"/>
-    <inertia ixx="2e-06" iyy="2e-06" izz="2e-06" ixy="0.0" iyz="-0.0" ixz="-0.0"/>
+    <origin xyz="-0.019999999999999934 3.893746217885482e-17 -0.012188268156424563" rpy="0 0 0"/>
+    <mass value="0.017408884194903936"/>
+    <inertia ixx="2e-06" iyy="2e-06" izz="2e-06" ixy="0.0" iyz="0.0" ixz="-0.0"/>
   </inertial>
   <visual>
@@ -100,7 +107,7 @@
   </visual>
   <collision>
-    <origin xyz="-0.1675 -0.0 -0.0291" rpy="0 0 0"/>
+    <origin xyz="0.0 0.0 0.0" rpy="0 0 0"/>
     <geometry>
-      <mesh filename="file://$(find bot_description)/meshes/caster_wheel_a_1.stl" scale="0.001 0.001 0.001"/>
+      <sphere radius="0.028"/>
     </geometry>
   </collision>
@@ -108,6 +115,6 @@
 <link name="camera_link_1">
   <inertial>
-    <origin xyz="0.00289127586298088 0.0010656513836692378 0.012889229339118194" rpy="0 0 0"/>
-    <mass value="0.006742869777511351"/>
+    <origin xyz="0.0033912758702940027 0.001065651333291926 0.012978229354270815" rpy="0 0 0"/>
+    <mass value="0.0011080639299913741"/>
     <inertia ixx="0.0" iyy="0.0" izz="0.0" ixy="-0.0" iyz="0.0" ixz="-0.0"/>
   </inertial>
@@ -128,10 +135,10 @@
 <link name="lidar_link_1">
   <inertial>
-    <origin xyz="-0.0006078599059984313 -0.00013002224629664804 0.014307180955488885" rpy="0 0 0"/>
-    <mass value="0.053104251406073145"/>
+    <origin xyz="-0.0006078599059954476 -0.00013002224628911718 0.014307180955489912" rpy="0 0 0"/>
+    <mass value="0.0531042514060907"/>
     <inertia ixx="2.4e-05" iyy="2.4e-05" izz="4.4e-05" ixy="0.0" iyz="-0.0" ixz="-0.0"/>
   </inertial>
   <visual>
-    <origin xyz="-0.115878 0.002021 -0.163831" rpy="0 0 0"/>
+    <origin xyz="-0.115878 0.002021 -0.164331" rpy="0 0 0"/>
     <geometry>
       <mesh filename="file://$(find bot_description)/meshes/lidar_link_1.stl" scale="0.001 0.001 0.001"/>
@@ -140,5 +147,5 @@
   </visual>
   <collision>
-    <origin xyz="-0.115878 0.002021 -0.163831" rpy="0 0 0"/>
+    <origin xyz="-0.115878 0.002021 -0.164331" rpy="0 0 0"/>
     <geometry>
       <mesh filename="file://$(find bot_description)/meshes/lidar_link_1.stl" scale="0.001 0.001 0.001"/>
@@ -174,5 +181,5 @@
 </joint>
 <joint name="lidar_joint" type="fixed">
-  <origin xyz="0.115878 -0.002021 0.163831" rpy="0 0 0"/>
+  <origin xyz="0.115878 -0.002021 0.164331" rpy="0 0 0"/>
   <parent link="base_link"/>
   <child link="lidar_link_1"/>
